Commit message: updated workspace

File: src/rotors_simulator/rotors_description/urdf/firefly.xacro (robot description, xacro)
@@ -27,5 +27,5 @@
   <xacro:property name="body_width" value="0.1" />
   <!-- [m] -->
-  <xacro:property name="body_height" value="0.06" />
+  <xacro:property name="body_height" value="1" />
   <!-- [m] -->
   <xacro:property name="mass_rotor" value="0.005" />
@@ -94,8 +94,8 @@
   <!-- CUSTOM EDITS BELOW -->
   <!--  -->
-  <!-- <xacro:camera_macro namespace="${namespace}" parent_link="${namespace}/base_link" camera_suffix="nadir" frame_rate="60.0" horizontal_fov="2" image_width="752" image_height="480" image_format="L8" min_distance="0.02" max_distance="50" noise_mean="0.0" noise_stddev="0.007" enable_visual="true">
+  <xacro:camera_macro namespace="${namespace}" parent_link="${namespace}/base_link" camera_suffix="nadir" frame_rate="60.0" horizontal_fov="2" image_width="752" image_height="480" image_format="L8" min_distance="0.02" max_distance="50" noise_mean="0.0" noise_stddev="0.007" enable_visual="true">
     <box size="0.05 0.05 0.02" />
     <origin xyz="0 0 ${-arm_length/4}" rpy="0 ${pi/2} 0" />
-  </xacro:camera_macro> -->
+  </xacro:camera_macro>
   <!-- <xacro:vi_sensor_depth_macro namespace="${namespace}" parent_link="${namespace}/base_link" camera_suffix="depth" frame_rate="30.0" max_range="10.0" enable_depth_camera_visual="true">
         <box size="0.05 0.05 0.02" />
